File: hardware/2.3/board_main/main.brd (EAGLE design)
At the start: 86.6 x 64.5 mm, 100 parts, among them IC2 LM2937, Q1 8MHz, Q2MMBF170-7-F BSS123, U1 L3G4200D, U11 MCP73831T-2DCI/OT, U2 STM32F103C6T6A, U3 LSM9DS0, X1 MINI-USB-32005-201

Commit message: common commit
Parts:
- removed C32: 4.7uF, resistor:C0805
Connections:
- removed net N$14: C32.1, U2.22
- net CAM_CLK: now also U2.22; no longer U2.45
- net GND: no longer C32.2
Routing:
- net CAM_CLK: track 66.8 -> 37.5 mm, vias 1 -> 0
- net +3V3: track 434.6 -> 421.7 mm
- net N$14: track 3.16 -> 0.00 mm
- net GND: track 598.3 -> 596.0 mm, vias 83 -> 82
- net SDA: track 101.4 -> 102.7 mm
- net SCL: track 92.7 -> 93.8 mm
- net USBDP: track 53.0 -> 54.1 mm
- net CAM_SI: track 47.7 -> 46.6 mm
- net USBDM: track 54.3 -> 55.1 mm
- net ADC8: track 31.8 -> 31.3 mm
