File: hardware/2.3/sensor_rgb/sensor.sch (EAGLE design)
At the start: 100 parts, among them IC2 LM2937, Q1 8MHz, Q2MMBF170-7-F BSS123, U1 L3G4200D, U11 MCP73831T-2DCI/OT, U2 STM32F103C6T6A, U3 LSM9DS0, X1 MINI-USB-32005-201

Commit message: common commit
Parts:
- removed BOOT: (no value), jumper:JP1E
- removed C20: 22p, resistor:C-EUC0805
- removed C21, C22: 18p, resistor:C-EUC0805
- removed C23, C32: 4.7uF, resistor:C-EUC0805
- removed C24: 220n, resistor:C-EUC0805
- removed C25, C26, C28, C29, C30, C31, C9: 100n, resistor:C-EUC0805
- removed C27: 10uF, resistor:C-EUC0805
- removed C7: 22uF, resistor:CPOL-EU153CLV-0505
- removed D1: (no value), diode:DIODE-SMB
- removed H1, H2: MOUNT-HOLE2.8, holes:MOUNT-HOLE2.8
- removed I2C_EXT, PROGRAMMING, UART: (no value), con-lstb:MA04-1
- removed IC2: LM2937, linear:LM2937
- removed IO1: DRV8834, yellow_car:DRV8834
- removed JP1: 2 or single CellLi-Pol, jumper:JP1E
- removed LED11: (no value), led:LEDCHIPLED_1206
- removed LED12: poweron, led:LEDCHIPLED_1206
- removed LED13: charging, led:LEDCHIPLED_1206
- removed Q1: 8MHz, crystal:CRYSTALCTS406
- removed Q2MMBF170-7-F: BSS123, transistor-small-signal:BSS123
- removed R19, R20, R21, R22, R24, R25: 4k7, resistor:R-EU_M0805
- removed R27, R28, R30, R32, R33, R44: 330, resistor:R-EU_M0805
- removed R45: 47k, resistor:R-EU_M0805
- removed RESET, USER: DTSM-6, switch-tact:DTSM-6
- removed S1: (no value), switch:255SB
- removed SV1: SERVO/PWM, con-lstb:MA03-1
- removed SV2: (no value), con-lsta:FE07-2
- removed U$3: APDS9950, my_parts:APDS9950
- removed U1: L3G4200D, my_parts:L3G4200D
- removed U11: MCP73831T-2DCI/OT, Microchip-MCP73831T-2DCI_OT:MCP73831T-2DCI/OT
- removed U2: STM32F103C6T6A, stm32f103_lqfp48:STM32F103C6T6A
- removed U3: LSM9DS0, SparkFun-DigitalIC:LSM9DS0
- removed X1: MINI-USB-32005-201, con-cypressindustries:MINI-USB-32005-201
- added H3, H4: MOUNT-HOLE2.8, holes:MOUNT-HOLE2.8
- added LED1, LED2, LED3, LED4, LED9: (no value), my_parts:LEDCHIPLED_1206
- added R11, R12: 330, resistor:R-EU_M0805
- added T5: (no value), transistor:BC857A-PNP-SOT23-BEC
- added U$10, U$8, U$9: APDS9950, my_parts:APDS9950
- C1: value 100n -> 10uF; device resistor:C-EUC1206 -> resistor:C-EUC0805
- C10, C12, C14, C6: value 10uF -> 100n
- C11, C15, C5: value 100n -> 10uF
- C16: value 22p -> 22uF; device resistor:C-EUC0805 -> resistor:CPOL-EU153CLV-0505
- C17: value 470n -> 100n
- C18: value 10n -> 10uF
- C2: value 10uF -> 100n; device resistor:C-EUC1206 -> resistor:C-EUC0805
- C3: value 10n -> 10uF; device resistor:C-EUC1206 -> resistor:C-EUC0805
- C4: value 1uF -> 100n; device resistor:C-EUC1206 -> resistor:C-EUC0805
- C8: value 22uF -> 100n; device resistor:CPOL-EU153CLV-0505 -> resistor:C-EUC0805
- LED5, LED6, LED7: device led:LEDCHIPLED_1206 -> my_parts:LEDCHIPLED_1206
- LED8: device led:LEDCHIPLED_1206 -> led:LED5MM
- R1: value 47k -> 4k7; device resistor:R-EU_M1206 -> resistor:R-EU_M0805
- R10, R16: value 10k -> 330
- R13, R14: value 4k7 -> 330
- R15: value 47k -> 330
- R17, R2, R3, R4, R5: value 47k -> 4k7
- R23: value 4k7 -> 22
- R6: value 0R USE ONLY FOR SINGLE CELL -> 4k7; device resistor:R-EU_M1206 -> resistor:R-EU_M0805
- R7, R8: value 22 -> 4k7
- R9: value 1k5 -> 330
- SV3: value TSL1401 CAMERA -> (none); device con-lsta:FE05-1 -> con-lsta:FE07-2
- U$1: value MICRO_METAL_GEAR_MOTOR -> APDS9950; device pololu:MICRO_METAL_GEAR_MOTOR -> my_parts:APDS9950
- U$2: value MICRO_METAL_GEAR_MOTOR -> APDS9950_EDGE; device pololu:MICRO_METAL_GEAR_MOTOR -> my_parts:APDS9950_EDGE
- U$7: value DSSCIRCUITS_PCA9544A -> APDS9950; device PCA9544A Breakout PCB:DSSCIRCUITS_PCA9544A -> my_parts:APDS9950
Connections:
- removed net ADC0: SV2.10, U2.PA0-WKUP
- removed net ADC1: SV2.9, U2.PA1
- removed net ADC2: SV2.8, U2.PA2
- removed net ADC3: SV2.7, U2.PA3
- removed net ADC4: SV2.5, U2.PA4
- removed net ADC5: SV2.4, U2.PA5
- removed net ADC6: SV2.3, U2.PA6
- removed net ADC7: SV2.2, U2.PA7
- removed net ADC8: SV2.6, U2.PB0
- removed net ADC9: U2.PB1
- removed net AENBL: IO1.NENBL/AENBL, U2.PB13
- removed net APHASE: IO1.M0/APHASE, U2.PB5
- removed net BATT: D1.C, JP1.2, R6.1, S1.O, S1.P
- removed net BENBL: IO1.STEP/BENBL, U2.PB14
- removed net BPHASE: IO1.DIR/BPHASE, U2.PA15
- removed net CAM_AO: SV3.3, U2.PB12
- removed net CAM_CLK: SV3.4, U2.PB8
- removed net CAM_SI: SV3.5, U2.PB10
- removed net IR_CONTROLL: SV2.1, U2.PA8
- removed net LED_1: R28.2, U2.PB15
- removed net M1: IO1.M1, U2.PB4
- removed net N$17: R44.2, U11.STAT
- removed net N$18: R17.1, R5.1, U3.DEN(G)
- removed net N$2 (its old number): IO1.AOUT2, U$1.P$2
- removed net N$22: C4.2, IO1.VINT
- removed net N$23: LED12.A, R27.2
- removed net N$26: Q2MMBF170-7-F.D, R2.1, SV1.3
- removed net N$33: LED11.A, R28.1
- removed net N$38: LED5.A, R26.1
- removed net N$39: LED6.A, R30.1
- removed net N$40: LED7.A, R32.1
- removed net N$41: LED8.A, R33.1
- removed net N$53: C14.1, LED13.A, R6.2, U11.VBAT
- removed net N$54: R10.1, U11.PROG
- removed net N$55: C20.2, R7.1, X1.2
- removed net N$56: C16.1, R8.1, X1.3
- removed net N$57: C13.1, D1.A, U11.VDD, X1.1
- removed net N$9 (its old number): IO1.NSLEEP, R1.2
- removed net OSCIN: C22.1, Q1.2, U2.PD0-OSC_IN
- removed net OSCOUT: C21.1, Q1.1, U2.PD1-OSC_OUT
- removed net RESET: C25.2, PROGRAMMING.1, R15.1, RESET.3, RESET.4, U2.NRST
- removed net SCL0: R19.1, U$3.SDA, U$7.SCL0
- removed net SCL1: R21.1, U$4.SDA, U$7.SCL1
- removed net SCL2: R23.1, U$5.SDA, U$7.SCL2
- removed net SCL3: R25.1, U$6.SDA, U$7.SCL3
- removed net SDA: I2C_EXT.4, R13.1, U$7.SDA, U1.SDA/SDI, U2.PB7, U3.SDA
- removed net SDA0: R18.1, U$3.SCL, U$7.SDA0
- removed net SDA1: R20.1, U$4.SCL, U$7.SDA1
- removed net SDA2: R22.1, U$5.SCL, U$7.SDA2
- removed net SDA3: R24.1, U$6.SCL, U$7.SDA3
- removed net SERVO: Q2MMBF170-7-F.G, R45.2, U2.PC13-TAMPER-RTC
- removed net SWCLK: PROGRAMMING.4, U2.PA14
- removed net SWDIO: PROGRAMMING.2, U2.PA13
- removed net UART_RX: U2.PA10, UART.2
- removed net UART_TX: U2.PA9, UART.3
- removed net USBDM: R7.2, U2.PA11
- removed net USBDP: R8.2, R9.2, U2.PA12
- removed net USER_KEY_1: R3.2, U2.PB9, USER.3
- removed net VCC: C1.1, C10.1, C2.1, C3.1, C7.+, C9.1, IC2.VI, IO1.VM, IO1.VM1, R1.1, R2.2, S1.S, SV1.2
- new net ADC0_: R8.1, SV3.10, U$10.SDA
- new net ADC1_: R7.1, SV3.9, U$9.SDA
- new net ADC2_: R6.1, SV3.8, U$8.SDA
- new net ADC3_: R5.1, SV3.7, U$7.SDA
- new net ADC4_: R4.1, SV3.5, U$6.SDA
- new net ADC5_: R3.1, SV3.4, U$5.SDA
- new net ADC6_: R2.1, SV3.3, U$4.SDA
- new net ADC7_: R1.1, SV3.2, U$1.SDA
- new net ADC8_: R17.1, SV3.6, U$2.SDA
- new net N$27: U$9.LDR, U$9.LEDK
- new net N$31: U$10.LDR, U$10.LEDK
- new net N$32: R26.1, T5.B
- net +3V3: now also C1.2, C10.2, C11.2, C12.2, C13.2, C14.2, C15.2, C16.+, C17.2, C18.2, C2.2, C3.2, C4.2, C5.2, C6.2, C8.2, R1.2, R10.1, R11.1, R12.1, R13.1, R14.1, R15.1, R16.1, R2.2, R3.2, R4.2, R5.2, R6.2, R7.2, R8.2, SV3.13, SV3.14, T5.E, U$1.LEDA, U$1.VDD, U$10.LEDA, U$10.VDD, U$2.LEDA, U$2.VDD, U$7.LEDA, U$8.LEDA, U$8.VDD, U$9.LEDA, U$9.VDD; no longer BOOT.1, C11.1, C12.1, C15.1, C26.2, C27.2, C28.2, C29.2, C30.2, C31.2, C5.1, C6.1, C8.+, I2C_EXT.2, IC2.VO, R13.2, R14.2, R15.2, R19.2, R20.2, R21.2, R22.2, R23.2, R24.2, R25.2, R26.2, R27.1, R3.1, R30.2, R32.2, R33.2, SV2.13, SV2.14, SV3.2, U$3.LEDA, U$3.VDD, U1.CS, U1.RSVDV@0, U1.VDD, U1.VDDIO, U2.VDDA, U2.VDD_1, U2.VDD_2, U2.VDD_3, U3.CS(G), U3.CS(XM), U3.VDD, U3.VDD_IO, UART.1
- net GND: now also C1.1, C10.1, C11.1, C12.1, C13.1, C14.1, C15.1, C16.-, C2.1, C3.1, C5.1, C6.1, C8.1, LED1.C, LED2.C, LED3.C, LED4.C, LED9.C, SV3.11, SV3.12, U$1.GND, U$10.GND, U$2.GND, U$8.GND, U$9.GND; no longer C1.2, C10.2, C11.2, C12.2, C13.2, C14.2, C15.2, C16.2, C2.2, C20.1, C21.2, C22.2, C23.1, C25.1, C26.1, C27.1, C28.1, C29.1, C30.1, C31.1, C32.2, C5.2, C6.2, C7.-, C8.-, C9.2, I2C_EXT.1, IC2.GND, IO1.ADECAY, IO1.AISEN, IO1.BDECAY, IO1.BISEN, IO1.CONFIG, IO1.GND, IO1.GND_PAD, JP1.1, LED11.C, LED12.C, PROGRAMMING.3, Q2MMBF170-7-F.S, R10.2, R4.2, R45.1, R5.2, RESET.1, RESET.2, SV1.1, SV2.11, SV2.12, SV3.1, U$3.GND, U$7.!INT0, U$7.!INT1, U$7.!INT2, U$7.!INT3, U$7.A0, U$7.A1, U$7.A2, U1.GND, U1.RSDVG@3, U1.RSVDG@0, U1.RSVDG@1, U1.RSVDG@2, U1.RSVDG@4, U1.SDO, U11.VSS, U2.PB2, U2.VSSA, U2.VSS_1, U2.VSS_2, U2.VSS_3, U3.GND, U3.SDO(G), U3.SDO(XM), UART.4, USER.1, USER.2, X1.5
- net N$1: now also R23.2, T5.C; no longer IO1.AOUT1, U$1.P$1
- net N$13: now also LED6.A, R14.2; no longer C24.1, U3.SETP
- net N$14: now also LED7.A, R15.2; no longer C32.1, U2.PB11
- net N$16: now also LED9.A, R16.2; no longer BOOT.2, R4.1, U2.BOOT0
- net N$19: now also R26.2, U$2.LDR, U$2.LEDK; no longer C18.2, R16.2, U1.PLL
- net N$20: now also U$7.LDR, U$7.LEDK; no longer C17.2, R16.1
- net N$24: now also U$8.LDR, U$8.LEDK; no longer LED13.C, R44.1
- net N$28: now also LED8.A, R23.1; no longer U$3.LDR, U$3.LEDK
- net N$3: now also LED1.A, R9.2; no longer IO1.BOUT1, U$2.P$1
- net N$4: now also U$1.LDR, U$1.LEDK; no longer IO1.BOUT2, U$2.P$2
- net N$5: now also LED2.A, R10.2; no longer C3.2, IO1.VCP
- net N$6: now also LED3.A, R11.2; no longer C23.2, U3.C1
- net N$7: now also LED4.A, R12.2; no longer C24.2, U3.SETC
- net N$8: now also LED5.A, R13.2; no longer IO1.AVREF, IO1.BVREF, IO1.VREFO
- net SCL: now also R18.1, SV3.1, U$1.SCL, U$10.SCL, U$2.SCL, U$4.SCL, U$5.SCL, U$6.SCL, U$8.SCL, U$9.SCL; no longer I2C_EXT.3, R14.1, U1.SCL, U2.PB6, U3.SCL
Other:
- note removed: "CONTROLL"
- note removed: "IMU - GYROSCOPE, ACCELEROMETER, MAGNETOMETER"
- note removed: "MCU - ARM CORTEX M3"
- note removed: "MOTOR DRIVER"
- note removed: "POWER SUPPLY"
- note removed: "rear sensor array"
- moved on the sheet: C1, C10, C11, C12, C13, C14, C15, C17, C18, C19, C2, C3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
