File: hardware/2.5/board_main/main.brd (EAGLE design)
At the start: 86.4 x 67.5 mm, 100 parts, among them IC2 LM2937, Q1 8MHz, Q2MMBF170-7-F BSS123, U1 L3G4200D, U11 MCP73831T-2DCI/OT, U2 STM32F103C6T6A, U3 LSM9DS0, X1 MINI-USB-32005-201

Commit message: common commit
Routing:
- net +3V3: track 431.0 -> 434.6 mm, vias 14 -> 15
- net GND: vias 86 -> 83
Other:
- board size 86.4 x 67.5 mm -> 86.6 x 64.5 mm
Changed lines of the file:
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@@
 <setting verticaltext="up"/>
 </settings>
-<grid distance="8" unitdist="mil" unit="mil" style="lines" multiple="1" display="yes" altdistance="0.025" altunitdist="inch" altunit="inch"/>
+<grid distance="8" unitdist="mil" unit="mil" style="lines" multiple="1" display="no" altdistance="0.025" altunitdist="inch" altunit="inch"/>
 <layers>
 <layer number="1" name="Top" color="4" fill="1" visible="yes" active="yes"/>
@@
 <board>
 <plain>
+<wire x1="8.7376" y1="1.27" x2="32.3342" y2="1.27" width="0.254" layer="20"/>
+<wire x1="67.7164" y1="1.27" x2="92.1004" y2="1.27" width="0.254" layer="20"/>
+<wire x1="93.726" y1="3.0226" x2="93.726" y2="65.786" width="0.254" layer="20"/>
+<wire x1="7.112" y1="65.786" x2="7.112" y2="2.9464" width="0.254" layer="20"/>
+<wire x1="93.726" y1="65.786" x2="77.47" y2="55.372" width="0.254" layer="20" curve="-70.595758"/>
+<wire x1="22.86" y1="55.372" x2="7.112" y2="65.786" width="0.254" layer="20" curve="-70.595758"/>
+<wire x1="22.86" y1="55.372" x2="25.4508" y2="55.372" width="0.254" layer="20"/>
+<wire x1="35.6362" y1="55.372" x2="66.3448" y2="55.4228" width="0.254" layer="20"/>
+<wire x1="75.8952" y1="55.372" x2="77.47" y2="55.372" width="0.254" layer="20"/>
+<wire x1="32.3342" y1="1.27" x2="67.7164" y2="1.27" width="0.254" layer="20" curve="-36"/>
+<wire x1="8.7376" y1="1.27" x2="7.112" y2="2.9464" width="0.254" layer="20" curve="-102.535931"/>
+<wire x1="93.726" y1="3.0226" x2="92.1004" y2="1.27" width="0.254" layer="20" curve="-102.535931"/>
+<wire x1="30.5562" y1="60.1472" x2="25.4508" y2="55.372" width="0.254" layer="20" curve="-70.595758"/>
+<wire x1="35.6362" y1="55.372" x2="30.5562" y2="60.1472" width="0.254" layer="20" curve="-70.595758"/>
+<wire x1="70.9422" y1="60.706" x2="66.3448" y2="55.4228" width="0.254" layer="20" curve="-70.595758"/>
+<wire x1="75.8952" y1="55.372" x2="70.9422" y2="60.706" width="0.254" layer="20" curve="-70.595758"/>
 <rectangle x1="47.8536" y1="31.496" x2="48.4632" y2="32.1056" layer="1" rot="R90"/>
 <rectangle x1="52.1208" y1="35.7632" x2="52.7304" y2="36.3728" layer="1" rot="R90"/>
@@
 <rectangle x1="52.324" y1="21.7424" x2="52.9336" y2="22.352" layer="1" rot="R90"/>
 <rectangle x1="48.0568" y1="17.6784" x2="48.6664" y2="18.288" layer="1" rot="R90"/>
-<wire x1="10.16" y1="57.0992" x2="31.0896" y2="57.0992" width="0.254" layer="20"/>
-<wire x1="69.4944" y1="57.0992" x2="91.0336" y2="57.0992" width="0.254" layer="20"/>
-<wire x1="93.472" y1="55.0672" x2="93.472" y2="-10.3632" width="0.254" layer="20"/>
-<wire x1="87.1728" y1="1.016" x2="68.2752" y2="1.016" width="0.254" layer="20"/>
-<wire x1="56.4896" y1="1.016" x2="44.5008" y2="1.016" width="0.254" layer="20"/>
-<wire x1="32.7152" y1="1.016" x2="13.0048" y2="1.016" width="0.254" layer="20"/>
-<wire x1="7.112" y1="-10.3632" x2="7.112" y2="55.0672" width="0.254" layer="20"/>
-<wire x1="69.4944" y1="57.0992" x2="31.0896" y2="57.0992" width="0.254" layer="20" curve="-19.03305"/>
-<wire x1="7.112" y1="55.0672" x2="10.16" y2="57.0992" width="0.254" layer="20" curve="-65.512796"/>
-<wire x1="91.0336" y1="57.0992" x2="93.472" y2="55.0672" width="0.254" layer="20" curve="-65.512796"/>
-<wire x1="7.112" y1="-10.3632" x2="13.0048" y2="1.016" width="0.254" layer="20" curve="-37.868997"/>
-<wire x1="87.1728" y1="1.016" x2="93.472" y2="-10.3632" width="0.254" layer="20" curve="-37.868997"/>
-<wire x1="62.1792" y1="-7.5184" x2="68.2752" y2="1.016" width="0.254" layer="20" curve="-37.868997"/>
-<wire x1="56.4896" y1="1.016" x2="62.1792" y2="-7.5184" width="0.254" layer="20" curve="-37.868997"/>
-<wire x1="32.7152" y1="1.016" x2="38.4048" y2="-7.5184" width="0.254" layer="20" curve="-37.868997"/>
-<wire x1="38.4048" y1="-7.5184" x2="44.5008" y2="1.016" width="0.254" layer="20" curve="-37.868997"/>
 </plain>
 <attributes>
@@
 <wire x1="74.0401625" y1="45.8478375" x2="74.7776" y2="45.1104" width="0.254" layer="1"/>
 <wire x1="74.7776" y1="45.1104" x2="75.184" y2="45.1104" width="0.254" layer="1"/>
-<via x="90.17" y="54.7624" extent="1-16" drill="0.6"/>
+<via x="87.122" y="55.5752" extent="1-16" drill="0.6"/>
 <wire x1="77.189759375" y1="39.9567875" x2="77.189759375" y2="40.004159375" width="0.254" layer="1"/>
 <wire x1="78.0288" y1="40.795828125" x2="77.189759375" y2="39.9567875" width="0.254" layer="1"/>
@@
 <vertex x="-1.4224" y="67.2592"/>
 <vertex x="102.2096" y="67.2592"/>
-<vertex x="102.8192" y="-14.8336"/>
-<vertex x="-0.8128" y="-14.8336"/>
+<vertex x="102.2096" y="-2.032"/>
+<vertex x="-1.4224" y="-2.032"/>
 </polygon>
 <polygon width="0.4064" layer="1">
 <vertex x="-6.2992" y="71.9328"/>
 <vertex x="104.2416" y="71.9328"/>
-<vertex x="104.8512" y="-19.5072"/>
-<vertex x="-5.6896" y="-19.5072"/>
+<vertex x="104.2416" y="-9.9568"/>
+<vertex x="-6.2992" y="-9.9568"/>
 </polygon>
 <contactref element="C32" pad="2"/>
@@
 <wire x1="73.548225" y1="46.2924" x2="73.9927875" y2="45.8478375" width="0.3048" layer="1"/>
 <via x="58.3692" y="42.8244" extent="1-16" drill="0.6"/>
-<via x="74.1172" y="54.5592" extent="1-16" drill="0.6"/>
-<via x="37.9984" y="3.0988" extent="1-16" drill="0.6"/>
-<via x="62.1792" y="3.0988" extent="1-16" drill="0.6"/>
 </signal>
 <signal name="VCC">
@@
 <contactref element="IO1" pad="19"/>
 <contactref element="IO1" pad="18"/>
+<wire x1="77.3378" y1="6.8084" x2="77.3378" y2="4.7162" width="0.3048" layer="1"/>
+<wire x1="77.3378" y1="4.7162" x2="76.584" y2="4.2164" width="0.3048" layer="1"/>
+<wire x1="76.6878" y1="6.8084" x2="76.6878" y2="4.0662" width="0.3048" layer="1"/>
 <wire x1="76.6878" y1="4.0662" x2="76.584" y2="4.2164" width="0.3048" layer="1"/>
 <contactref element="C1" pad="1"/>
@@
 <wire x1="32.1056" y1="2.6416" x2="19.1008" y2="2.6416" width="1.27" layer="1"/>
 <wire x1="19.1008" y1="2.6416" x2="17.3736" y2="4.3688" width="1.27" layer="1"/>
-<wire x1="76.6878" y1="6.8084" x2="76.6878" y2="4.3202" width="0.4064" layer="1"/>
-<wire x1="76.6878" y1="4.3202" x2="76.584" y2="4.2164" width="0.4064" layer="1"/>
-<wire x1="77.3378" y1="6.8084" x2="77.3378" y2="4.9702" width="0.4064" layer="1"/>
-<wire x1="77.3378" y1="4.9702" x2="76.584" y2="4.2164" width="0.4064" layer="1"/>
 </signal>
 <signal name="+3V3">
@@
 <wire x1="78.486" y1="52.324" x2="81.026" y2="52.324" width="0.6096" layer="16"/>
 <wire x1="81.026" y1="52.324" x2="81.407" y2="51.943" width="0.6096" layer="16"/>
+<wire x1="80.684" y1="53.594" x2="80.684" y2="52.666" width="0.254" layer="1"/>
+<wire x1="80.684" y1="52.666" x2="81.407" y2="51.943" width="0.254" layer="1"/>
 <via x="81.407" y="51.943" extent="1-16" drill="0.6"/>
+<wire x1="81.534" y1="51.816" x2="81.407" y2="51.943" width="0.254" layer="1"/>
 <wire x1="58.2676" y1="52.1716" x2="58.2676" y2="49.6316" width="0.6096" layer="16"/>
+<via x="57.404" y="40.132" extent="1-16" drill="0.6"/>
 <wire x1="68.326" y1="32.004" x2="72.136" y2="32.004" width="0.4064" layer="16"/>
 <wire x1="77.531009375" y1="39.615540625" x2="77.613940625" y2="39.615540625" width="0.254" layer="1"/>
@@
 <wire x1="77.613940625" y1="39.615540625" x2="77.613940625" y2="39.022859375" width="0.254" layer="1"/>
 <wire x1="77.613940625" y1="39.022859375" x2="78.0288" y2="38.608" width="0.254" layer="1"/>
+<wire x1="60.3504" y1="39.8272" x2="60.3504" y2="39.624" width="0.4064" layer="16"/>
 <wire x1="60.3504" y1="39.624" x2="60.96" y2="39.0144" width="0.4064" layer="16"/>
 <wire x1="60.96" y1="39.0144" x2="66.04" y2="39.0144" width="0.4064" layer="16"/>
@@
 <wire x1="40.8432" y1="47.0256" x2="41.2496" y2="46.6192" width="0.4064" layer="16"/>
 <wire x1="83.42205625" y1="43.495009375" x2="88.859409375" y2="43.495009375" width="0.254" layer="1"/>
+<wire x1="78.0288" y1="38.608" x2="77.4192" y2="38.608" width="0.254" layer="16"/>
+<wire x1="77.4192" y1="38.608" x2="76.8096" y2="37.9984" width="0.254" layer="16"/>
+<wire x1="76.8096" y1="37.9984" x2="76.8096" y2="32.1056" width="0.254" layer="16"/>
+<wire x1="89.3572" y1="43.942" x2="90.6272" y2="42.672" width="0.254" layer="1"/>
+<wire x1="90.6272" y1="42.672" x2="90.6272" y2="41.4392" width="0.254" layer="1"/>
 <wire x1="90.6272" y1="41.4392" x2="90.6644" y2="41.402" width="0.254" layer="1"/>
 <via x="78.4352" y="32.3088" extent="1-16" drill="0.6"/>
@@
 <wire x1="81.28" y1="49.00413125" x2="80.60225625" y2="48.3263875" width="0.254" layer="1"/>
 <wire x1="84.455" y1="51.8922" x2="84.9376" y2="51.4096" width="0.6096" layer="16"/>
-<wire x1="60.3504" y1="39.624" x2="60.3504" y2="40.4368" width="0.4064" layer="16"/>
+<wire x1="57.404" y1="40.132" x2="57.8104" y2="40.132" width="0.4064" layer="16"/>
+<wire x1="57.8104" y1="40.132" x2="58.1152" y2="39.8272" width="0.4064" layer="16"/>
+<wire x1="58.1152" y1="39.8272" x2="60.3504" y2="39.8272" width="0.4064" layer="16"/>
+<wire x1="60.3504" y1="39.8272" x2="60.3504" y2="40.4368" width="0.4064" layer="16"/>
 <wire x1="60.3504" y1="40.4368" x2="60.96" y2="41.0464" width="0.4064" layer="16"/>
 <wire x1="60.96" y1="41.0464" x2="63.1952" y2="41.0464" width="0.4064" layer="16"/>
@@
 <wire x1="55.0672" y1="36.9824" x2="55.0672" y2="37.9324" width="0.3048" layer="1"/>
 <wire x1="55.0672" y1="37.9324" x2="54.8488" y2="38.1508" width="0.3048" layer="1"/>
-<wire x1="80.684" y1="53.594" x2="80.684" y2="52.666" width="0.6096" layer="1"/>
-<wire x1="80.684" y1="52.666" x2="81.407" y2="51.943" width="0.6096" layer="1"/>
-<wire x1="90.6272" y1="41.4392" x2="90.6272" y2="42.7228" width="0.6096" layer="1"/>
-<wire x1="90.6272" y1="42.7228" x2="89.3572" y2="43.9928" width="0.6096" layer="1"/>
-<wire x1="76.8096" y1="32.1056" x2="76.8096" y2="37.3888" width="0.4064" layer="16"/>
-<wire x1="76.8096" y1="37.3888" x2="78.0288" y2="38.608" width="0.4064" layer="16"/>
 </signal>
 <signal name="SCL">
