File: hardware/main_board_custom_bridge_v2/main.sch (EAGLE design)
At the start: 66 parts, among them IC2 LM2937, Q1 8MHz, U11 MCP73831T-2DCI/OT, U2 STM32F103C6T6A, U3 LSM9DS0, X1 MINI-USB-32005-201

Commit message: common
Parts:
- removed C13, C14: 10uF, resistor:C-EUC0805
- removed C3: 10n, resistor:C-EUC1206
- removed C4: 1uF, resistor:C-EUC1206
- removed IO1: DRV8834, yellow_car:DRV8834
- removed LED13: charging, led:LEDCHIPLED_1206
- removed PROGRAMMING: (no value), con-lstb:MA04-1
- removed R17, R5: 47k, resistor:R-EU_M0805
- removed R44: 330, resistor:R-EU_M0805
- removed U$1, U$2: MICRO_METAL_GEAR_MOTOR, pololu:MICRO_METAL_GEAR_MOTOR
- removed U11: MCP73831T-2DCI/OT, Microchip-MCP73831T-2DCI_OT:MCP73831T-2DCI/OT
- added IC1: MCP1703CB, linear:MCP1703CB
- added Q2MMBF170-7-F1, Q2MMBF170-7-F2, Q2MMBF170-7-F3, Q2MMBF170-7-F4, Q2MMBF170-7-F5, Q2MMBF170-7-F6: BSS123, transistor-small-signal:BSS123
- added R11, R12, R16, R18, R19, R20, R21: 4k7, resistor:R-EU_M0805
- added SV4: MOTOR_B_PWM, con-lstb:MA03-1
- added SV5: MOTOR_A_PWM, con-lstb:MA03-1
- added SV6: MOTOR_B_PHASE_INV, con-lstb:MA03-1
- added SV7: MOTOR_A_PHASE_INV, con-lstb:MA03-1
- added SV8: MOTOR_A_PHASE, con-lstb:MA03-1
- added SV9: MOTOR_B_PHASE, con-lstb:MA03-1
- C1: value 100n -> 10uF; device resistor:C-EUC1206 -> resistor:C-EUC0805
- C2: value 10uF -> 100n; device resistor:C-EUC1206 -> resistor:C-EUC0805
- R1: value 47k -> 4k7; device resistor:R-EU_M1206 -> resistor:R-EU_M0805
- R10: value 10k -> 4k7
- R6: value 0R USE ONLY FOR SINGLE CELL -> 4k7; device resistor:R-EU_M1206 -> resistor:R-EU_M0805
Connections:
- removed net N$17: R44.2, U11.STAT
- removed net N$18: R17.1, R5.1, U3.DEN(G)
- removed net N$22: C4.2, IO1.VINT
- removed net N$24: LED13.C, R44.1
- removed net N$53: C14.1, LED13.A, R6.2, U11.VBAT
- removed net N$54: R10.1, U11.PROG
- removed net N$9: IO1.NSLEEP, R1.2
- new net +5V: C1.1, IC1.VO, R1.2, R10.2, R11.2, R18.2, R20.2, R21.2
- net +3V3: now also R12.1, R6.1; no longer R17.2
- net AENBL: now also Q2MMBF170-7-F1.G, R12.2; no longer IO1.NENBL/AENBL
- net APHASE: now also Q2MMBF170-7-F3.G, R16.2; no longer IO1.M0/APHASE
- net BATT: no longer D1.C, R6.1
- net BENBL: now also Q2MMBF170-7-F2.G, R6.2; no longer IO1.STEP/BENBL
- net BPHASE: now also Q2MMBF170-7-F4.G, R19.2; no longer IO1.DIR/BPHASE
- net GND: now also IC1.GND, Q2MMBF170-7-F1.S, Q2MMBF170-7-F2.S, Q2MMBF170-7-F3.S, Q2MMBF170-7-F4.S, Q2MMBF170-7-F5.S, Q2MMBF170-7-F6.S, R16.1, R19.1, SV4.1, SV5.1, SV6.1, SV7.1, SV8.1, SV9.1; no longer C13.2, C14.2, C4.1, IO1.ADECAY, IO1.AISEN, IO1.BDECAY, IO1.BISEN, IO1.CONFIG, IO1.GND, IO1.GND_PAD, PROGRAMMING.3, R10.2, R5.2, U11.VSS
- net M1: no longer IO1.M1
- net N$1: now also Q2MMBF170-7-F5.D, R20.1, SV8.3; no longer IO1.AOUT1, U$1.P$1
- net N$2: now also Q2MMBF170-7-F4.D, Q2MMBF170-7-F6.G, R18.1, SV6.3; no longer IO1.AOUT2, U$1.P$2
- net N$3: now also Q2MMBF170-7-F1.D, R11.1, SV5.3; no longer IO1.BOUT1, U$2.P$1
- net N$4: now also Q2MMBF170-7-F2.D, R1.1, SV4.3; no longer IO1.BOUT2, U$2.P$2
- net N$5: now also Q2MMBF170-7-F3.D, Q2MMBF170-7-F5.G, R10.1, SV7.3; no longer C3.2, IO1.VCP
- net N$57: no longer C13.1, U11.VDD
- net N$8: now also Q2MMBF170-7-F6.D, R21.1, SV9.3; no longer IO1.AVREF, IO1.BVREF, IO1.VREFO
- net RESET: no longer PROGRAMMING.1
- net SWCLK: no longer PROGRAMMING.4
- net SWDIO: no longer PROGRAMMING.2
- net VCC: now also D1.C, IC1.VI, SV4.2, SV5.2, SV6.2, SV7.2, SV8.2, SV9.2; no longer C1.1, C3.1, IO1.VM, IO1.VM1, R1.1
Other:
- moved on the sheet: C1, C10, C11, C12, C16, C2, C20, C7, C8, C9, D1, IC2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
