File: hardware/main_board_v3/main.brd (EAGLE design)
At the start: 87.5 x 74 mm, 87 parts, among them IC1 24AA32ASN, IC2 LM2937, IC3 VNH3SP30, IC4 78L05F, IC5 VNH3SP30, Q1 8MHz, Q2 BSS123, Q3 BSS123, Q4 BSS123, Q5 BSS123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

Commit message: board rev 3
Parts:
- added Q8, Q9: BSS123, transistor-small-signal:SOT23
- added R24, R25, R26: 4k7, resistor:M0805
- added U$1, U$2, U$3, U$4, U$5, U$6, U$7, U$8, U$9: FIDUCIAL, adafruit:FIDUCIAL_1MM
- moved X4 0.61 mm to (70.4, 11.2)
Connections:
- new net MOTOR_ENABLE: Q9.1, R24.1, U4.38
- new net M_ENABLE: IC3.10, IC3.6, IC5.10, IC5.6, Q8.3, R25.2
- new net N$17: Q8.1, Q9.3, R26.2
- net +5V: now also R25.1, R26.1
- net BPHASE: now also U4.54; no longer U4.50
- net GND: now also Q8.2, Q9.2, R24.2
Routing:
- net M_ENABLE: track 0.00 -> 59.1 mm, vias 0 -> 4
- net MOTOR_ENABLE: track 0.00 -> 34.5 mm, vias 0 -> 4
- net GND: track 630.7 -> 646.0 mm, vias 68 -> 70
- net +5V: track 68.6 -> 78.9 mm, vias 1 -> 2
- net N$17: track 0.00 -> 4.83 mm
- net APHASE: track 20.9 -> 22.3 mm
- net IR_CONTROLL: track 27.9 -> 29.2 mm
- net N$20: track 6.66 -> 5.63 mm
- net BPHASE: track 38.3 -> 39.2 mm
- net N$14: track 42.9 -> 43.7 mm
- net BENBL: track 59.3 -> 58.6 mm
- net APHASE2: track 30.5 -> 30.0 mm
