File: hardware/main_board_v3/main.sch (EAGLE design)
At the start: 87 parts, among them IC1 24AA32ASN, IC2 LM2937, IC3 VNH3SP30, IC4 78L05F, IC5 VNH3SP30, Q1 8MHz, Q2 BSS123, Q3 BSS123, Q4 BSS123, Q5 BSS123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

Commit message: board rev 3
Parts:
- added Q8, Q9: BSS123, transistor-small-signal:BSS123
- added R24, R25, R26: 4k7, resistor:R-EU_M0805
- added U$1, U$2, U$3, U$4, U$5, U$6, U$7, U$8, U$9: FIDUCIAL, adafruit:FIDUCIAL
Connections:
- new net MOTOR_ENABLE: Q9.G, R24.1, U4B.PC7
- new net M_ENABLE: IC3.DIAGA, IC3.DIAGB, IC5.DIAGA, IC5.DIAGB, Q8.D, R25.2
- new net N$17: Q8.G, Q9.D, R26.2
- net +5V: now also R25.1, R26.1
- net BPHASE: now also U4B.PD2; no longer U4B.PA15
- net GND: now also Q8.S, Q9.S, R24.2
Other:
- moved on the sheet: Q4, Q5, Q6, R10, R11, R12, R2, R5, R6
